File: _autosave-new project.kicad_sch (KiCad schematic)
At the start: 4 parts, among them J1 LED 0.170amps, J2 Tractive Battery

Commit message: Wiring Done
Parts:
- J1: footprint Resistor_SMD:R_0201_0603Metric -> Connector_Molex:Molex_Micro-Fit_3.0_43650-0200_1x02_P3.00mm_Horizontal
- R1: footprint Resistor_SMD:R_0201_0603Metric -> Capacitor_SMD:C_0603_1608Metric
Changed lines of the file:
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@@
 			)
 		)
-		(property "Footprint" "Resistor_SMD:R_0201_0603Metric"
+		(property "Footprint" "Connector_Molex:Molex_Micro-Fit_3.0_43650-0200_1x02_P3.00mm_Horizontal"
 			(at 35.56 110.49 0)
 			(effects
@@
 			)
 		)
-		(property "Footprint" "Resistor_SMD:R_0201_0603Metric"
+		(property "Footprint" "Capacitor_SMD:C_0603_1608Metric"
 			(at 74.93 94.488 90)
 			(effects
