File: new project.kicad_sch (KiCad schematic)
At the start: 4 parts

Commit message: Autosave
Parts:
- J1: renamed from J?; footprint Resistor_SMD:R_0201_0603Metric -> Connector_Molex:Molex_Micro-Fit_3.0_43650-0200_1x02_P3.00mm_Horizontal
- R1: renamed from R?; footprint Resistor_SMD:R_0201_0603Metric -> Capacitor_SMD:C_0603_1608Metric
- U1: renamed from U?; footprint IXCP10M90S:IXCP10M90S -> Package_TO_SOT_SMD:TO-252-2
- gave numbers to parts that had none: 1
Changed lines of the file:
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@@
 		(on_board yes)
 		(dnp no)
-		(property "Reference" "J?"
+		(property "Reference" "J2"
 			(at 56.515 107.95 0)
 			(effects
@@
 			(project ""
 				(path "/077e92cf-3ae1-46e9-bd7c-3f2e84892e92"
-					(reference "J?")
+					(reference "J2")
 					(unit 1)
 				)
@@
 		(dnp no)
 		(fields_autoplaced yes)
-		(property "Reference" "J?"
+		(property "Reference" "J1"
 			(at 36.195 105.41 0)
 			(effects
@@
 			)
 		)
-		(property "Footprint" "Resistor_SMD:R_0201_0603Metric"
+		(property "Footprint" "Connector_Molex:Molex_Micro-Fit_3.0_43650-0200_1x02_P3.00mm_Horizontal"
 			(at 35.56 110.49 0)
 			(effects
@@
 			(project ""
 				(path "/077e92cf-3ae1-46e9-bd7c-3f2e84892e92"
-					(reference "J?")
+					(reference "J1")
 					(unit 1)
 				)
@@
 		(dnp no)
 		(fields_autoplaced yes)
-		(property "Reference" "U?"
+		(property "Reference" "U1"
 			(at 52.07 98.4249 0)
 			(effects
@@
 			)
 		)
-		(property "Footprint" "IXCP10M90S:IXCP10M90S"
+		(property "Footprint" "Package_TO_SOT_SMD:TO-252-2"
 			(at 39.37 100.33 0)
 			(effects
@@
 			(project ""
 				(path "/077e92cf-3ae1-46e9-bd7c-3f2e84892e92"
-					(reference "U?")
+					(reference "U1")
 					(unit 1)
 				)
@@
 		(dnp no)
 		(fields_autoplaced yes)
-		(property "Reference" "R?"
+		(property "Reference" "R1"
 			(at 74.93 86.36 90)
 			(effects
@@
 			)
 		)
-		(property "Footprint" "Resistor_SMD:R_0201_0603Metric"
+		(property "Footprint" "Capacitor_SMD:C_0603_1608Metric"
 			(at 74.93 94.488 90)
 			(effects
@@
 			(project ""
 				(path "/077e92cf-3ae1-46e9-bd7c-3f2e84892e92"
-					(reference "R?")
-					(unit 1)
-				)
+					(reference "R1")
+					(unit 1)
+				)
