File: breakout board/breakout board.kicad_sch (KiCad schematic)
At the start: 3 parts, among them J1 Conn_01x07_Pin, J2 Conn_01x07_Pin, U1 MCP2518FD-xQBB

Commit message: work
Connections:
- net at J2.1 (Pin_1): now also U1.15 (VSS), U1.7 (VSS); no longer U1.8 (~{INT1}/GPIO1)
- net at J2.2 (Pin_2): now also U1.6 (OSC1); no longer U1.9 (~{INT0}/GPIO0/XSTBY)
- net at J2.3 (Pin_3): now also U1.5 (OSC2); no longer U1.4 (~{INT})
- net at J2.4 (Pin_4): now also U1.4 (~{INT}); no longer U1.3 (CLKO/SOF)
- net at J2.5 (Pin_5): now also U1.3 (CLKO/SOF); no longer U1.1 (TXCAN)
- net at J2.7 (Pin_7): now also U1.1 (TXCAN); no longer U1.14 (VDD)
- net at J1.1 (Pin_1): now also U1.8 (~{INT1}/GPIO1); no longer U1.11 (SDI)
- net at J1.2 (Pin_2): now also U1.9 (~{INT0}/GPIO0/XSTBY); no longer U1.12 (SDO)
- net at J1.3 (Pin_3): now also U1.10 (SCK); no longer U1.13 (~{CS})
- net at J1.4 (Pin_4): now also U1.11 (SDI); no longer U1.10 (SCK)
- net at J1.5 (Pin_5): now also U1.12 (SDO); no longer U1.5 (OSC2)
- net at J1.6 (Pin_6): now also U1.13 (~{CS}); no longer U1.6 (OSC1)
- new net: J1.7 (Pin_7), U1.14 (VDD)
